Commit message: Replace placeholder URDF dimensions with measured values; base_link at ground level

File: ros2_ws/src/mecanum_description/urdf/mecanum_robot.urdf.xacro (robot description, xacro)
@@ -1,18 +1,63 @@
 <?xml version="1.0"?>
 <robot name="mecanum_robot" xmlns:xacro="http://www.ros.org/wiki/xacro">
-  <xacro:property name="lx" value="0.1"/>
-  <xacro:property name="ly" value="0.1"/>
-  <xacro:property name="wheel_radius" value="0.0483"/>
-  <xacro:property name="wheel_width" value="0.03"/>
-  <xacro:property name="base_length" value="0.25"/>
-  <xacro:property name="base_width" value="0.22"/>
-  <xacro:property name="base_height" value="0.10"/>
-<xacro:macro name="wheel" params="prefix x_offset y_offset">
+  <!-- ==============================================================
+       FRAME CONVENTION
+       base_link : point on the floor below the centroid of the
+                   200x200mm wheel-contact square. X fwd, Y left,
+                   Z up, z=0 at the floor.
+       Every property below traces to a Station.
+       ============================================================== -->
+  <!-- Station 3: wheels -->
+  <xacro:property name="wheel_radius_geom" value="0.0484"/>
+  <xacro:property name="wheel_width"       value="0.0435"/>
+  <xacro:property name="lx" value="0.100"/>
+  <xacro:property name="ly" value="0.100"/>
+  <!-- Station 4: frame -->
+  <xacro:property name="frame_length"    value="0.259"/>
+  <xacro:property name="frame_width"     value="0.141"/>
+  <xacro:property name="frame_thickness" value="0.00305"/>
+  <xacro:property name="frame_bottom_z"  value="0.070"/>
+  <!-- Station 5: lidar. Scan axis = midpoint of the cylindrical body.
+       0.190(Deck2) + 0.015(standoff) + 0.023(base) + half of 0.015(cyl) = 0.2355 -->
+  <xacro:property name="lidar_base_length" value="0.055"/>
+  <xacro:property name="lidar_base_width"  value="0.055"/>
+  <xacro:property name="lidar_base_height" value="0.023"/>
+  <xacro:property name="lidar_cyl_radius"  value="0.0253"/>
+  <xacro:property name="lidar_cyl_height"  value="0.015"/>
+  <xacro:property name="lidar_cyl_half_height" value="0.0075"/>
+  <xacro:property name="lidar_x" value="0.1275"/>
+  <xacro:property name="lidar_y" value="0.0"/>
+  <xacro:property name="lidar_z" value="0.2355"/>
+  <!-- Station 6: IMU -->
+  <xacro:property name="imu_x" value="-0.046"/>
+  <xacro:property name="imu_y" value="0.005"/>
+  <xacro:property name="imu_z" value="0.2084"/>
+  <xacro:property name="imu_yaw" value="${pi}"/>
+  <xacro:property name="imu_board_x" value="0.021"/>
+  <xacro:property name="imu_board_y" value="0.016"/>
+  <xacro:property name="imu_board_z" value="0.002"/>
+  <!-- Derived convenience values (not new measurements) -->
+  <xacro:property name="frame_centre_z"
+    value="${frame_bottom_z + frame_thickness/2}"/>
+  <xacro:property name="lidar_base_offset_z"
+    value="${-(lidar_cyl_half_height + lidar_base_height/2)}"/>
+  <material name="frame_grey"><color rgba="0.55 0.56 0.58 1.0"/></material>
+  <material name="wheel_black"><color rgba="0.12 0.12 0.14 1.0"/></material>
+  <material name="lidar_black"><color rgba="0.18 0.18 0.20 1.0"/></material>
+  <material name="lidar_teal"><color rgba="0.36 0.88 0.85 1.0"/></material>
+  <material name="imu_blue"><color rgba="0.15 0.35 0.75 1.0"/></material>
+  <link name="base_link">
+    <visual>
+      <origin xyz="0 0 ${frame_centre_z}" rpy="0 0 0"/>
+      <geometry><box size="${frame_length} ${frame_width} ${frame_thickness}"/></geometry>
+      <material name="frame_grey"/>
+    </visual>
+  </link>
+  <xacro:macro name="mecanum_wheel" params="prefix x_sign y_sign">
     <link name="${prefix}_wheel_link">
       <visual>
-        <origin xyz="0 0 0" rpy="1.5708 0 0"/>
-        <geometry>
-          <cylinder radius="${wheel_radius}" length="${wheel_width}"/>
-        </geometry>
+        <origin xyz="0 0 0" rpy="${pi/2} 0 0"/>
+        <geometry><cylinder radius="${wheel_radius_geom}" length="${wheel_width}"/></geometry>
+        <material name="wheel_black"/>
       </visual>
     </link>
@@ -20,20 +65,22 @@
       <parent link="base_link"/>
       <child link="${prefix}_wheel_link"/>
-      <origin xyz="${x_offset} ${y_offset} -0.05" rpy="0 0 0"/>
+      <origin xyz="${x_sign * lx} ${y_sign * ly} ${wheel_radius_geom}" rpy="0 0 0"/>
       <axis xyz="0 1 0"/>
     </joint>
   </xacro:macro>
-  <link name="base_link">
-    <visual>
-      <geometry>
-        <box size="${base_length} ${base_width} ${base_height}"/>
-      </geometry>
-    </visual>
-  </link>
+  <xacro:mecanum_wheel prefix="front_left"  x_sign="1"  y_sign="1"/>
+  <xacro:mecanum_wheel prefix="front_right" x_sign="1"  y_sign="-1"/>
+  <xacro:mecanum_wheel prefix="rear_left"   x_sign="-1" y_sign="1"/>
+  <xacro:mecanum_wheel prefix="rear_right"  x_sign="-1" y_sign="-1"/>
   <link name="lidar_link">
     <visual>
-      <geometry>
-        <cylinder radius="0.03" length="0.04"/>
-      </geometry>
+      <origin xyz="0 0 0" rpy="0 0 0"/>
+      <geometry><cylinder radius="${lidar_cyl_radius}" length="${lidar_cyl_height}"/></geometry>
+      <material name="lidar_teal"/>
+    </visual>
+    <visual>
+      <origin xyz="0 0 ${lidar_base_offset_z}" rpy="0 0 0"/>
+      <geometry><box size="${lidar_base_length} ${lidar_base_width} ${lidar_base_height}"/></geometry>
+      <material name="lidar_black"/>
     </visual>
   </link>
@@ -41,9 +88,17 @@
     <parent link="base_link"/>
     <child link="lidar_link"/>
-    <origin xyz="0.20 0.0 0.15" rpy="0 0 0"/>
+    <origin xyz="${lidar_x} ${lidar_y} ${lidar_z}" rpy="0 0 0"/>
   </joint>
-  <xacro:wheel prefix="front_left" x_offset="${lx}" y_offset="${ly}"/>
-  <xacro:wheel prefix="front_right" x_offset="${lx}" y_offset="${-ly}"/>
-  <xacro:wheel prefix="rear_left" x_offset="${-lx}" y_offset="${ly}"/>
-  <xacro:wheel prefix="rear_right" x_offset="${-lx}" y_offset="${-ly}"/>
+  <link name="imu_link">
+    <visual>
+      <origin xyz="0 0 0" rpy="0 0 0"/>
+      <geometry><box size="${imu_board_x} ${imu_board_y} ${imu_board_z}"/></geometry>
+      <material name="imu_blue"/>
+    </visual>
+  </link>
+  <joint name="imu_joint" type="fixed">
+    <parent link="base_link"/>
+    <child link="imu_link"/>
+    <origin xyz="${imu_x} ${imu_y} ${imu_z}" rpy="0 0 ${imu_yaw}"/>
+  </joint>
 </robot>

Commit message: Make URDF physics-ready for Gazebo: inertia + collision on all links
Add reusable box_inertial and cylinder_inertial xacro macros that compute the inertia tensor from mass and geometry (standard solid-body formulas), so tensors always match the shapes.

Every link now has mass, inertia, and collision:
- base_link: 3.0 kg. Inertia uses a realistic mass envelope (0.13 m tall box centered at z=0.135) rather than the 3 mm visual plate, so the stacked-robot mass distribution simulates stably instead of behaving like a thin sheet. Visual/collision keep the real plate.
- four wheels: 0.08 kg each. Cylinder inertial passed a rpy=pi/2 origin so the axial term lands on the y spin axis, matching the wheel joint axis.
- lidar_link, imu_link: token 0.01 kg inertials (their real mass is folded into base_link) plus simple box collision, kept small to avoid solver instability on tiny fixed links.

Masses from kitchen-scale measurements (chassis+decks+wheels 2.6 kg,wheels 80 g each, plus lidar/pi/stm32/battery and mounting hardware,rounded to 3.0 kg for base_link). Verified: xacro expands cleanly,7 links each with 1 inertial and 1 collision.

File: ros2_ws/src/mecanum_description/urdf/mecanum_robot.urdf.xacro (robot description, xacro)
@@ -1,4 +1,31 @@
 <?xml version="1.0"?>
 <robot name="mecanum_robot" xmlns:xacro="http://www.ros.org/wiki/xacro">
+<!-- ==============================================================
+       INERTIA MACROS
+       Compute the inertia tensor from mass + geometry so the numbers
+       always match the shapes. Box and cylinder formulas.
+       ============================================================== -->
+  <xacro:macro name="box_inertial" params="mass x y z *origin">
+    <inertial>
+      <xacro:insert_block name="origin"/>
+      <mass value="${mass}"/>
+      <inertia
+        ixx="${(1/12) * mass * (y*y + z*z)}"
+        iyy="${(1/12) * mass * (x*x + z*z)}"
+        izz="${(1/12) * mass * (x*x + y*y)}"
+        ixy="0" ixz="0" iyz="0"/>
+    </inertial>
+  </xacro:macro>
+  <xacro:macro name="cylinder_inertial" params="mass radius length *origin">
+    <inertial>
+      <xacro:insert_block name="origin"/>
+      <mass value="${mass}"/>
+      <inertia
+        ixx="${(1/12) * mass * (3*radius*radius + length*length)}"
+        iyy="${(1/12) * mass * (3*radius*radius + length*length)}"
+        izz="${(1/2) * mass * radius*radius}"
+        ixy="0" ixz="0" iyz="0"/>
+    </inertial>
+  </xacro:macro>
   <!-- ==============================================================
        FRAME CONVENTION
@@ -47,5 +74,5 @@
   <material name="lidar_teal"><color rgba="0.36 0.88 0.85 1.0"/></material>
   <material name="imu_blue"><color rgba="0.15 0.35 0.75 1.0"/></material>
-  <link name="base_link">
+<link name="base_link">
     <visual>
       <origin xyz="0 0 ${frame_centre_z}" rpy="0 0 0"/>
@@ -53,6 +80,13 @@
       <material name="frame_grey"/>
     </visual>
+    <collision>
+      <origin xyz="0 0 ${frame_centre_z}" rpy="0 0 0"/>
+      <geometry><box size="${frame_length} ${frame_width} ${frame_thickness}"/></geometry>
+    </collision>
+    <xacro:box_inertial mass="3.0" x="${frame_length}" y="${frame_width}" z="0.13">
+      <origin xyz="0 0 0.135" rpy="0 0 0"/>
+    </xacro:box_inertial>
   </link>
-  <xacro:macro name="mecanum_wheel" params="prefix x_sign y_sign">
+<xacro:macro name="mecanum_wheel" params="prefix x_sign y_sign">
     <link name="${prefix}_wheel_link">
       <visual>
@@ -61,4 +95,11 @@
         <material name="wheel_black"/>
       </visual>
+      <collision>
+        <origin xyz="0 0 0" rpy="${pi/2} 0 0"/>
+        <geometry><cylinder radius="${wheel_radius_geom}" length="${wheel_width}"/></geometry>
+      </collision>
+      <xacro:cylinder_inertial mass="0.08" radius="${wheel_radius_geom}" length="${wheel_width}">
+        <origin xyz="0 0 0" rpy="${pi/2} 0 0"/>
+      </xacro:cylinder_inertial>
     </link>
     <joint name="${prefix}_wheel_joint" type="continuous">
@@ -84,4 +125,11 @@
       <material name="lidar_black"/>
     </visual>
+    <collision>
+      <origin xyz="0 0 ${lidar_base_offset_z}" rpy="0 0 0"/>
+      <geometry><box size="${lidar_base_length} ${lidar_base_width} ${lidar_base_height}"/></geometry>
+    </collision>
+    <xacro:box_inertial mass="0.01" x="${lidar_base_length}" y="${lidar_base_width}" z="${lidar_base_height}">
+      <origin xyz="0 0 0" rpy="0 0 0"/>
+    </xacro:box_inertial>
   </link>
   <joint name="lidar_joint" type="fixed">
@@ -96,4 +144,11 @@
       <material name="imu_blue"/>
     </visual>
+    <collision>
+      <origin xyz="0 0 0" rpy="0 0 0"/>
+      <geometry><box size="${imu_board_x} ${imu_board_y} ${imu_board_z}"/></geometry>
+    </collision>
+    <xacro:box_inertial mass="0.01" x="${imu_board_x}" y="${imu_board_y}" z="${imu_board_z}">
+      <origin xyz="0 0 0" rpy="0 0 0"/>
+    </xacro:box_inertial>
   </link>
   <joint name="imu_joint" type="fixed">
